File: driver/_autosave-driver.sch (KiCad schematic (older format))
At the start: 24 parts, among them J1 Screw_Terminal_01x04, J2 Screw_Terminal_01x04, J3 Conn_01x03_Female, J4 Conn_01x03_Female, J5 Barrel_Jack, SW1 SW_SPDT, SW2 SW_SPDT, SW3 SW_SPDT, U1 NCP1117ST50T3G

Commit message: Added connector project, mostly laid out driver.
Parts:
- C5: footprint Capacitor_SMD:C_0201_0603Metric_Pad0.64x0.40mm_HandSolder -> Capacitor_SMD:C_0805_2012Metric_Pad1.18x1.45mm_HandSolder; Digi-Key Part Number 1276-1013-1-ND -> 478-08056D104KAT2ACT-ND
- D1: value 1N4007 -> S1MB-13-F; footprint Diode_THT:D_DO-41_SOD81_P10.16mm_Horizontal -> Diode_SMD:D_SMB; Digi-Key Part Number (none) -> S1MB-FDICT-ND
Connections:
- net at XA1.D12: now also SW1.1 (A); no longer SW1.3 (C)
Other:
- moved on the sheet: H2, H3, H4, J1, J2, SW1
