File: connector/_autosave-connector.kicad_pcb (KiCad board)
At the start: 2 copper layers, 20 x 24.5 mm, 6 parts, among them J1 Conn_01x04_Female, J2 Conn_01x04

Commit message: Fit test passed, panelized boards. Ready to order soon
Other:
- board text added: "Silent Dripper Connector"
- board text added: "v1.0.0 (Feb '21) Support - dev@esologic.com"
Changed lines of the file:
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@@
   (general
     (thickness 1.6)
-    (drawings 18)
+    (drawings 20)
     (tracks 14)
     (zones 0)
@@
     (visible_elements FFFFFF7F)
     (pcbplotparams
-      (layerselection 0x010fc_ffffffff)
-      (usegerberextensions false)
-      (usegerberattributes true)
-      (usegerberadvancedattributes true)
-      (creategerberjobfile true)
+      (layerselection 0x010f0_ffffffff)
+      (usegerberextensions true)
+      (usegerberattributes false)
+      (usegerberadvancedattributes false)
+      (creategerberjobfile false)
       (excludeedgelayer true)
       (linewidth 0.100000)
@@
       (viasonmask false)
       (mode 1)
-      (useauxorigin false)
+      (useauxorigin true)
       (hpglpennumber 1)
       (hpglpenspeed 20)
@@
       (outputformat 1)
       (mirror false)
-      (drillshape 1)
+      (drillshape 0)
       (scaleselection 1)
-      (outputdirectory ""))
+      (outputdirectory "connector-gerbers/"))
   )
   (net 0 "")
@@
       (effects (font (size 1 1) (thickness 0.15)))
     )
-    (pad 1 thru_hole roundrect (at 0 0) (size 1.7 1.95) (drill 0.95) (layers *.Cu *.Mask) (roundrect_rratio 0.147059)
+    (pad 1 thru_hole roundrect (at 0 0) (size 1.7 1.95) (drill 0.95) (layers *.Cu *.Mask) (roundrect_rratio 0.1470588235294118)
       (net 1 /Motor_Phase_A1_Red))
     (pad 2 thru_hole oval (at 2.5 0) (size 1.7 1.95) (drill 0.95) (layers *.Cu *.Mask)
@@
     )
   )
+  (gr_text "Silent Dripper Connector" (at 99.9906 99.5934) (layer B.SilkS)
+    (effects (font (size 0.8 0.8) (thickness 0.2)) (justify mirror))
+  )
+  (gr_text "v1.0.0 (Feb '21)\nSupport - dev@esologic.com" (at 99.9906 104.4194) (layer B.SilkS)
+    (effects (font (size 0.8 0.8) (thickness 0.2)) (justify mirror))
+  )
   (gr_line (start 96.25 101.725) (end 103.75 101.725) (layer Dwgs.User) (width 0.2))
